Commit message: Send idle flag back to controller when cartesian_pose control finished

File: resources/franka_panda.urdf (robot description, URDF)
Before this commit: robot franka_panda, 8 links, 7 joints
Links:
- link link7: geometry collision mesh filename=collision/finger.stl; collision mesh filename=collision/finger.stl

Commit message: Use collada graphics instead of obj

File: resources/franka_panda.urdf (robot description, URDF)
Before this commit: robot franka_panda, 8 links, 7 joints
Links:
- link link0: geometry collision mesh filename=collision/link0.stl; visual mesh filename=visual/link0.dae
- link link1: geometry collision mesh filename=collision/link1.stl; visual mesh filename=visual/link1.dae
- link link2: geometry collision mesh filename=collision/link2.stl; visual mesh filename=visual/link2.dae
- link link3: geometry collision mesh filename=collision/link3.stl; visual mesh filename=visual/link3.dae
- link link4: geometry collision mesh filename=collision/link4.stl; visual mesh filename=visual/link4.dae
- link link5: geometry collision mesh filename=collision/link5.stl; visual mesh filename=visual/link5.dae
- link link6: geometry collision mesh filename=collision/link6.stl; visual mesh filename=visual/link6.dae
- link link7: geometry collision mesh filename=collision/finger.stl; collision mesh filename=collision/finger.stl
